Commit message: FIC Control Studio 6.1.0

File: fic_ws/src/menagerie/model/Franka_FR3/URDF/Franka_FR3.urdf (robot description, URDF)
Before this commit: robot fr3, 17 links, 16 joints
Links:
- link fr3_link0: mass None -> 2.82067
- link fr3_link1: mass None -> 2.92747
- link fr3_link2: mass None -> 2.93554
- link fr3_link3: mass None -> 2.2449
- link fr3_link4: mass None -> 2.6156
- link fr3_link5: mass None -> 2.32712
- link fr3_link6: mass None -> 1.81704
- link fr3_link7: mass None -> 0.627143

File: fic_ws/src/menagerie/model/Pendulum/URDF/Pendulum.urdf (robot description, URDF)
Before this commit: robot pendulum, 3 links, 2 joints
Links:
- removed link mass
- added link ee_link
- added link world
- link base_link: geometry 
- link pole: mass 0.5 -> 1.51; geometry visual cylinder length=0.5 radius=0.02; visual sphere radius=0.05
Joints:
- removed joint ee_link
- removed joint hinge
- added joint Actuator1: type revolute, parent base_link, child pole, axis 0 1 0, limit lower=-3.14159 upper=3.14159 effort=39.0 velocity=10.0
- added joint base_joint: type fixed, parent world, child base_link, origin xyz=0 0 0.6
- added joint ee_joint: type fixed, parent pole, child ee_link, origin xyz=0 0 0.5
